Commit message: - rendered anymal - bug fix is needed

File: res/r2d2/r2d2.urdf (robot description, URDF)
Before this commit: robot physics, 16 links, 15 joints
Links:
- link base_link: geometry collision cylinder length=0.6 radius_=0.17; visual cylinder length=0.6 radius_=0.2
- link gripper_pole: geometry collision cylinder length=0.2 radius_=.01; visual cylinder length=0.2 radius_=.01
- link head: geometry collision sphere radius_=0.16; visual sphere radius_=0.16
- link left_back_wheel: geometry collision cylinder length=.1 radius_=0.035; visual cylinder length=.1 radius_=0.035
- link left_front_wheel: geometry collision cylinder length=.1 radius_=0.035; visual cylinder length=.1 radius_=0.035
- link right_back_wheel: geometry collision cylinder length=.1 radius_=0.035; visual cylinder length=.1 radius_=0.035
- link right_front_wheel: geometry collision cylinder length=.1 radius_=0.035; visual cylinder length=.1 radius_=0.035
