Commit message: - odesim  - set generalized velocity

File: res/2DRobotArm/robot.urdf (robot description, URDF)
Before this commit: robot 2DrobotArm, 4 links, 3 joints
Links:
- link link1: mass None -> 1

Commit message: - odesim  - added prismatic joint (not finished)  - edited capler urdf

File: res/2DRobotArm/robot.urdf (robot description, URDF)
Before this commit: robot 2DrobotArm, 4 links, 3 joints
Links:
- link link1: mass 1 -> None

File: res/Capler/robot.urdf (robot description, URDF)
Before this commit: robot caplerleg, 9 links, 8 joints
Links:
- removed link FOOT_CONTACT
- removed link FOOT_MOUNT
- removed link FOOT_SENSOR
- added link FOOT, mass 0.15; collision sphere radius=0.032; visual cylinder length=0.03 radius=0.015
Joints:
- removed joint MOUNT_TO_SENSOR
- removed joint SENSOR_TO_FOOT
- removed joint SHANK_TO_MOUNT
- added joint SHANK_TO_FOOT: type fixed, parent SHANK, child FOOT, origin xyz=0.0 -0.0228 -0.236 rpy=0.0 0.0 0.0
