Commit message: - bullet articulated system linear momentum getter error fixed

File: res/Singlebody/robot.urdf (robot description, URDF)
Before this commit: robot anymal, 1 links, 0 joints
Links:
- link base: mass 21.39 -> 10

Commit message: - debugging ode articulated system

File: res/Singlebody/robot.urdf (robot description, URDF)
Before this commit: robot singlebody, 1 links, 0 joints
Links:
- link base: geometry collision box size=1 1 1; visual box size=1 1 1

Commit message: - ode articulated system bug fixed. (mass position)

File: res/Singlebody/robot.urdf (robot description, URDF)
Before this commit: robot singlebody, 1 links, 0 joints
Links:
- link base: geometry collision box size=1 1 5; visual box size=1 1 5
