Commit message: - BtMb momentum debugged.

File: res/Multibody/robot.urdf (robot description, URDF)
Before this commit: robot anymal, 5 links, 4 joints
Links:
- removed link LF_FOOT_MOUNT
- removed link LF_HIP
- removed link LF_SHANK
- removed link LF_THIGH
- added link bar, mass 10; collision box size=1 0.2 0.2; visual box size=1 0.2 0.2
- link base: mass 21.39 -> 10; geometry collision box size=1 1 1; visual box size=1 1 1
Joints:
- removed joint LF_ANKLE_JOINT
- removed joint LF_HAA
- removed joint LF_HFE
- removed joint LF_KFE
- added joint revolute: type revolute, parent base, child bar, origin xyz=0.0 0.0 0.7, axis 0 0 1, limit lower=-6.28 upper=6.28 effort=80 velocity=15
