Commit message: - ode articulated system. now body frame = COM frame

File: res/ANYmal-nomesh/robot.urdf (robot description, URDF)
Before this commit: robot anymal, 18 links, 17 joints
Joints:
- joint LF_HFE: origin xyz=0.0585                    0.0315                    0.0 -> xyz=0.0585 0.0315 0.0
