Commit message: - anymal pd control test result updated

File: res/ANYmal-energy/robot.urdf (robot description, URDF)
Before this commit: robot anymal, 18 links, 17 joints
Joints:
- joint LF_HAA: limit effort=80 velocity=15 -> effort=0 velocity=15
- joint LF_HFE: limit effort=80 velocity=15 -> effort=0 velocity=15
- joint LF_KFE: limit effort=80 velocity=15 -> effort=0 velocity=15
- joint LH_HAA: limit effort=80 velocity=15 -> effort=0 velocity=15
- joint LH_HFE: limit effort=80 velocity=15 -> effort=0 velocity=15
- joint LH_KFE: limit effort=80 velocity=15 -> effort=0 velocity=15
- joint RF_HAA: limit effort=80 velocity=15 -> effort=0 velocity=15
- joint RF_HFE: limit effort=80 velocity=15 -> effort=0 velocity=15
- joint RF_KFE: limit effort=80 velocity=15 -> effort=0 velocity=15
- joint RH_HAA: limit effort=80 velocity=15 -> effort=0 velocity=15
- joint RH_HFE: limit effort=80 velocity=15 -> effort=0 velocity=15
- joint RH_KFE: limit effort=80 velocity=15 -> effort=0 velocity=15
