Commit message: - ANYmal-energy-benchmark bullet URDF and ode-rai-dart URDF edited - added BtMbBenchmark profile option

File: res/ANYmal-energy-benchmark/bullet/robot.urdf (robot description, URDF)
Before this commit: robot anymal, 18 links, 17 joints
Links:
- link LF_FOOT_MOUNT: geometry visual sphere radius=0.03
- link LF_HIP: geometry visual cylinder length=0.08 radius=0.04
- link LF_SHANK: geometry visual cylinder length=0.19 radius=0.015
- link LF_THIGH: geometry visual cylinder length=0.08 radius=0.04
- link LH_FOOT_MOUNT: geometry visual sphere radius=0.03
- link LH_HIP: geometry visual cylinder length=0.08 radius=0.04
- link LH_SHANK: geometry visual cylinder length=0.19 radius=0.015
- link LH_THIGH: geometry visual cylinder length=0.08 radius=0.04
- link RF_FOOT_MOUNT: geometry visual sphere radius=0.03
- link RF_HIP: geometry visual cylinder length=0.08 radius=0.04
- link RF_SHANK: geometry visual cylinder length=0.19 radius=0.015
- link RF_THIGH: geometry visual cylinder length=0.08 radius=0.04
- link RH_FOOT_MOUNT: geometry visual sphere radius=0.03
- link RH_HIP: geometry visual cylinder length=0.08 radius=0.04
- link RH_SHANK: geometry visual cylinder length=0.19 radius=0.015
- link RH_THIGH: geometry visual cylinder length=0.08 radius=0.04
- link base: geometry visual box size=0.531 0.232 0.26
- link imu_link: geometry visual box size=0.058 0.058 0.022
Joints:
- joint LF_HAA: limit effort=0 velocity=15 -> (none); type revolute -> continuous
- joint LF_HFE: limit effort=0 velocity=15 -> (none); origin xyz=0.0585                    0.0315                    0.0 -> xyz=0.0585 0.0315 0.0; type revolute -> continuous
- joint LF_KFE: limit effort=0 velocity=15 -> (none); type revolute -> continuous
- joint LH_HAA: limit effort=0 velocity=15 -> (none); type revolute -> continuous
- joint LH_HFE: limit effort=0 velocity=15 -> (none); origin xyz=-0.0585                    0.0315                    0.0 -> xyz=-0.0585 0.0315 0.0; type revolute -> continuous
- joint LH_KFE: limit effort=0 velocity=15 -> (none); type revolute -> continuous
- joint RF_HAA: limit effort=0 velocity=15 -> (none); type revolute -> continuous
- joint RF_HFE: limit effort=0 velocity=15 -> (none); type revolute -> continuous
- joint RF_KFE: limit effort=0 velocity=15 -> (none); type revolute -> continuous
- joint RH_HAA: limit effort=0 velocity=15 -> (none); type revolute -> continuous
- joint RH_HFE: limit effort=0 velocity=15 -> (none); type revolute -> continuous
- joint RH_KFE: limit effort=0 velocity=15 -> (none); type revolute -> continuous

File: res/ANYmal-energy-benchmark/ode-rai-dart/robot.urdf (robot description, URDF)
Before this commit: robot anymal, 18 links, 17 joints
Links:
- link LF_FOOT_MOUNT: geometry visual sphere radius=0.03
- link LF_HIP: geometry visual cylinder length=0.08 radius=0.04
- link LF_SHANK: geometry visual cylinder length=0.19 radius=0.015
- link LF_THIGH: geometry visual cylinder length=0.08 radius=0.04
- link LH_FOOT_MOUNT: geometry visual sphere radius=0.03
- link LH_HIP: geometry visual cylinder length=0.08 radius=0.04
- link LH_SHANK: geometry visual cylinder length=0.19 radius=0.015
- link LH_THIGH: geometry visual cylinder length=0.08 radius=0.04
- link RF_FOOT_MOUNT: geometry visual sphere radius=0.03
- link RF_HIP: geometry visual cylinder length=0.08 radius=0.04
- link RF_SHANK: geometry visual cylinder length=0.19 radius=0.015
- link RF_THIGH: geometry visual cylinder length=0.08 radius=0.04
- link RH_FOOT_MOUNT: geometry visual sphere radius=0.03
- link RH_HIP: geometry visual cylinder length=0.08 radius=0.04
- link RH_SHANK: geometry visual cylinder length=0.19 radius=0.015
- link RH_THIGH: geometry visual cylinder length=0.08 radius=0.04
- link base: geometry visual box size=0.531 0.232 0.26
- link imu_link: geometry visual box size=0.058 0.058 0.022
Joints:
- joint LF_HAA: limit effort=80 velocity=15 -> (none)
- joint LF_HFE: limit effort=80 velocity=15 -> (none); origin xyz=0.0585 0.0315 0.0 -> xyz=0.0585                    0.0315                    0.0
- joint LF_KFE: limit effort=80 velocity=15 -> (none)
- joint LH_HAA: limit effort=80 velocity=15 -> (none)
- joint LH_HFE: limit effort=80 velocity=15 -> (none); origin xyz=-0.0585                    0.0315                    0.0 -> xyz=-0.0585 0.0315 0.0
- joint LH_KFE: limit effort=80 velocity=15 -> (none)
- joint RF_HAA: limit effort=80 velocity=15 -> (none)
- joint RF_HFE: limit effort=80 velocity=15 -> (none); origin xyz=0.0585                    -0.0315                    0.0 -> xyz=0.0585 -0.0315 0.0
- joint RF_KFE: limit effort=80 velocity=15 -> (none)
- joint RH_HAA: limit effort=80 velocity=15 -> (none)
- joint RH_HFE: limit effort=80 velocity=15 -> (none); origin xyz=-0.0585                    -0.0315                    0.0 -> xyz=-0.0585 -0.0315 0.0
- joint RH_KFE: limit effort=80 velocity=15 -> (none)
