Commit message: - ANYmal energy benchmark mujoco urdf fixed - ANYmal-PD-benchmark URDF path changed - MJC disable contact setter (setWorldContactFlag) - ODE continuous joint

File: res/ANYmal-PD-benchmark/bullet/robot.urdf (robot description, URDF)
Before this commit: robot anymal, 28 links, 26 joints
Links:
- removed link LF_FOOT_0
- removed link LF_FOOT_MOUNT_0
- removed link LF_FOOT_SENSOR_0
- removed link LF_HIP_0
- removed link LF_SHANK_0
- removed link LF_THIGH_0
- removed link LH_FOOT_0
- removed link LH_FOOT_MOUNT_0
- removed link LH_FOOT_SENSOR_0
- removed link LH_HIP_0
- removed link LH_SHANK_0
- removed link LH_THIGH_0
- removed link RF_FOOT_0
- removed link RF_FOOT_MOUNT_0
- removed link RF_FOOT_SENSOR_0
- removed link RF_HIP_0
- removed link RF_SHANK_0
- removed link RF_THIGH_0
- removed link RH_FOOT_0
- removed link RH_FOOT_MOUNT_0
- removed link RH_FOOT_SENSOR_0
- removed link RH_HIP_0
- removed link RH_SHANK_0
- removed link RH_THIGH_0
- removed link base_0
- removed link ground
- removed link imu_link_0
- removed link world
- added link LF_FOOT_MOUNT, mass 0.1922685; collision sphere radius=0.03; visual sphere radius=0.03
- added link LF_HIP, mass 1.1064; collision cylinder length=0.08 radius=0.04; visual cylinder length=0.08 radius=0.04
- added link LF_SHANK, mass 0.318; collision cylinder length=0.19 radius=0.015; visual cylinder length=0.19 radius=0.015
- added link LF_THIGH, mass 1.51; collision cylinder length=0.08 radius=0.04; visual cylinder length=0.08 radius=0.04
- added link LH_FOOT_MOUNT, mass 0.1922685; collision sphere radius=0.03; visual sphere radius=0.03
- added link LH_HIP, mass 1.1064; collision cylinder length=0.08 radius=0.04; visual cylinder length=0.08 radius=0.04
- added link LH_SHANK, mass 0.318; collision cylinder length=0.19 radius=0.015; visual cylinder length=0.19 radius=0.015
- added link LH_THIGH, mass 1.51; collision cylinder length=0.08 radius=0.04; visual cylinder length=0.08 radius=0.04
- added link RF_FOOT_MOUNT, mass 0.1922685; collision sphere radius=0.03; visual sphere radius=0.03
- added link RF_HIP, mass 1.1064; collision cylinder length=0.08 radius=0.04; visual cylinder length=0.08 radius=0.04
- added link RF_SHANK, mass 0.318; collision cylinder length=0.19 radius=0.015; visual cylinder length=0.19 radius=0.015
- added link RF_THIGH, mass 1.51; collision cylinder length=0.08 radius=0.04; visual cylinder length=0.08 radius=0.04
- added link RH_FOOT_MOUNT, mass 0.1922685; collision sphere radius=0.03; visual sphere radius=0.03
- added link RH_HIP, mass 1.1064; collision cylinder length=0.08 radius=0.04; visual cylinder length=0.08 radius=0.04
- added link RH_SHANK, mass 0.318; collision cylinder length=0.19 radius=0.015; visual cylinder length=0.19 radius=0.015
- added link RH_THIGH, mass 1.51; collision cylinder length=0.08 radius=0.04; visual cylinder length=0.08 radius=0.04
- added link base, mass 21.39; collision box size=0.531 0.232 0.26; visual box size=0.531 0.232 0.26
- added link imu_link, mass 0.05; collision box size=0.058 0.058 0.022; visual box size=0.058 0.058 0.022
Joints:
- removed joint LF_ANKLE_JOINT_0
- removed joint LF_HAA_0
- removed joint LF_HFE_0
- removed joint LF_KFE_0
- removed joint LF_MOUNT_TO_SENSOR_0
- removed joint LF_SENSOR_TO_FOOT_0
- removed joint LH_ANKLE_JOINT_0
- removed joint LH_HAA_0
- removed joint LH_HFE_0
- removed joint LH_KFE_0
- removed joint LH_MOUNT_TO_SENSOR_0
- removed joint LH_SENSOR_TO_FOOT_0
- removed joint RF_ANKLE_JOINT_0
- removed joint RF_HAA_0
- removed joint RF_HFE_0
- removed joint RF_KFE_0
- removed joint RF_MOUNT_TO_SENSOR_0
- removed joint RF_SENSOR_TO_FOOT_0
- removed joint RH_ANKLE_JOINT_0
- removed joint RH_HAA_0
- removed joint RH_HFE_0
- removed joint RH_KFE_0
- removed joint RH_MOUNT_TO_SENSOR_0
- removed joint RH_SENSOR_TO_FOOT_0
- removed joint base_to_world_0
- removed joint imu_joint_0
- added joint LF_ANKLE_JOINT: type fixed, parent LF_SHANK, child LF_FOOT_MOUNT, origin xyz=0.0 -0.016 -0.31 rpy=0.323 0.549 0
- added joint LF_HAA: type revolute, parent base, child LF_HIP, origin xyz=0.2629 0.115 0.0, axis 1 0 0, limit lower=-6.28 upper=6.28 effort=80 velocity=15
- added joint LF_HFE: type revolute, parent LF_HIP, child LF_THIGH, origin xyz=0.0585 0.0315 0.0, axis 0 1 0, limit lower=-6.28 upper=6.28 effort=80 velocity=15
- added joint LF_KFE: type revolute, parent LF_THIGH, child LF_SHANK, origin xyz=0.0 0.111 -0.25, axis 0 1 0, limit lower=-6.28 upper=6.28 effort=80 velocity=15
- added joint LH_ANKLE_JOINT: type fixed, parent LH_SHANK, child LH_FOOT_MOUNT, origin xyz=-0.0 -0.016 -0.31 rpy=0.323 -0.549 0
- added joint LH_HAA: type revolute, parent base, child LH_HIP, origin xyz=-0.2629 0.115 0.0, axis 1 0 0, limit lower=-6.28 upper=6.28 effort=80 velocity=15
- added joint LH_HFE: type revolute, parent LH_HIP, child LH_THIGH, origin xyz=-0.0585                    0.0315                    0.0, axis 0 1 0, limit lower=-6.28 upper=6.28 effort=80 velocity=15
- added joint LH_KFE: type revolute, parent LH_THIGH, child LH_SHANK, origin xyz=-0.0 0.111 -0.25, axis 0 1 0, limit lower=-6.28 upper=6.28 effort=80 velocity=15
- added joint RF_ANKLE_JOINT: type fixed, parent RF_SHANK, child RF_FOOT_MOUNT, origin xyz=0.0 0.016 -0.31 rpy=-0.323 0.549 0
- added joint RF_HAA: type revolute, parent base, child RF_HIP, origin xyz=0.2629 -0.115 0.0, axis 1 0 0, limit lower=-6.28 upper=6.28 effort=80 velocity=15
- added joint RF_HFE: type revolute, parent RF_HIP, child RF_THIGH, origin xyz=0.0585                    -0.0315                    0.0, axis 0 1 0, limit lower=-6.28 upper=6.28 effort=80 velocity=15
- added joint RF_KFE: type revolute, parent RF_THIGH, child RF_SHANK, origin xyz=0.0 -0.111 -0.25, axis 0 1 0, limit lower=-6.28 upper=6.28 effort=80 velocity=15
- added joint RH_ANKLE_JOINT: type fixed, parent RH_SHANK, child RH_FOOT_MOUNT, origin xyz=-0.0 0.016 -0.31 rpy=-0.323 -0.549 0
- added joint RH_HAA: type revolute, parent base, child RH_HIP, origin xyz=-0.2629 -0.115 0.0, axis 1 0 0, limit lower=-6.28 upper=6.28 effort=80 velocity=15
- added joint RH_HFE: type revolute, parent RH_HIP, child RH_THIGH, origin xyz=-0.0585                    -0.0315                    0.0, axis 0 1 0, limit lower=-6.28 upper=6.28 effort=80 velocity=15
- added joint RH_KFE: type revolute, parent RH_THIGH, child RH_SHANK, origin xyz=-0.0 -0.111 -0.25, axis 0 1 0, limit lower=-6.28 upper=6.28 effort=80 velocity=15
- added joint imu_joint: type fixed, parent base, child imu_link, origin xyz=0.0245 -0.04255 0.1857 rpy=3.14159265359 0 0
