Commit message: - atlas contact benchmark fixed - mujoco contact visualization

File: res/benchmark/Atlas-contact-benchmark/ode-rai-dart/robot.urdf (robot description, URDF)
Before this commit: robot drc_skeleton, 44 links, 43 joints
Links:
- link l_lglut: geometry visual mesh filename=l_lglut.stl
- link l_uglut: geometry visual mesh filename=l_uglut.stl
- link r_lglut: geometry visual mesh filename=r_lglut.stl
- link r_uglut: geometry visual mesh filename=r_uglut.stl
