Commit message: - atlas test modified. (control to stand)

File: res/benchmark/Atlas-contact-benchmark/bullet/robot.urdf (robot description, URDF)
Before this commit: robot drc_skeleton, 44 links, 43 joints
Links:
- link l_foot: geometry collision box size=0.5 0.15 0.05; visual mesh filename=l_foot.stl
- link r_foot: geometry collision box size=0.5 0.15 0.05; visual mesh filename=r_foot.stl

File: res/benchmark/Atlas-contact-benchmark/mujoco/robot1.urdf (robot description, URDF)
Before this commit: robot drc_skeleton, 46 links, 44 joints
Links:
- link l_foot_0: geometry collision box size=0.5 0.2 0.05; visual mesh filename=l_foot.stl
- link r_foot_0: geometry collision box size=0.5 0.2 0.05; visual mesh filename=r_foot.stl

File: res/benchmark/Atlas-contact-benchmark/mujoco/robot16.urdf (robot description, URDF)
Before this commit: robot drc_skeleton, 706 links, 704 joints
Links:
- link l_foot_0: geometry collision box size=0.5 0.2 0.05; visual mesh filename=l_foot.stl
- link l_foot_1: geometry collision box size=0.5 0.2 0.05; visual mesh filename=l_foot.stl
- link l_foot_10: geometry collision box size=0.5 0.2 0.05; visual mesh filename=l_foot.stl
- link l_foot_11: geometry collision box size=0.5 0.2 0.05; visual mesh filename=l_foot.stl
- link l_foot_12: geometry collision box size=0.5 0.2 0.05; visual mesh filename=l_foot.stl
- link l_foot_13: geometry collision box size=0.5 0.2 0.05; visual mesh filename=l_foot.stl
- link l_foot_14: geometry collision box size=0.5 0.2 0.05; visual mesh filename=l_foot.stl
- link l_foot_15: geometry collision box size=0.5 0.2 0.05; visual mesh filename=l_foot.stl
- link l_foot_2: geometry collision box size=0.5 0.2 0.05; visual mesh filename=l_foot.stl
- link l_foot_3: geometry collision box size=0.5 0.2 0.05; visual mesh filename=l_foot.stl
- link l_foot_4: geometry collision box size=0.5 0.2 0.05; visual mesh filename=l_foot.stl
- link l_foot_5: geometry collision box size=0.5 0.2 0.05; visual mesh filename=l_foot.stl
- link l_foot_6: geometry collision box size=0.5 0.2 0.05; visual mesh filename=l_foot.stl
- link l_foot_7: geometry collision box size=0.5 0.2 0.05; visual mesh filename=l_foot.stl
- link l_foot_8: geometry collision box size=0.5 0.2 0.05; visual mesh filename=l_foot.stl
- link l_foot_9: geometry collision box size=0.5 0.2 0.05; visual mesh filename=l_foot.stl
- link r_foot_0: geometry collision box size=0.5 0.2 0.05; visual mesh filename=r_foot.stl
- link r_foot_1: geometry collision box size=0.5 0.2 0.05; visual mesh filename=r_foot.stl
- link r_foot_10: geometry collision box size=0.5 0.2 0.05; visual mesh filename=r_foot.stl
- link r_foot_11: geometry collision box size=0.5 0.2 0.05; visual mesh filename=r_foot.stl
- link r_foot_12: geometry collision box size=0.5 0.2 0.05; visual mesh filename=r_foot.stl
- link r_foot_13: geometry collision box size=0.5 0.2 0.05; visual mesh filename=r_foot.stl
- link r_foot_14: geometry collision box size=0.5 0.2 0.05; visual mesh filename=r_foot.stl
- link r_foot_15: geometry collision box size=0.5 0.2 0.05; visual mesh filename=r_foot.stl
- link r_foot_2: geometry collision box size=0.5 0.2 0.05; visual mesh filename=r_foot.stl
- link r_foot_3: geometry collision box size=0.5 0.2 0.05; visual mesh filename=r_foot.stl
- link r_foot_4: geometry collision box size=0.5 0.2 0.05; visual mesh filename=r_foot.stl
- link r_foot_5: geometry collision box size=0.5 0.2 0.05; visual mesh filename=r_foot.stl
- link r_foot_6: geometry collision box size=0.5 0.2 0.05; visual mesh filename=r_foot.stl
- link r_foot_7: geometry collision box size=0.5 0.2 0.05; visual mesh filename=r_foot.stl
- link r_foot_8: geometry collision box size=0.5 0.2 0.05; visual mesh filename=r_foot.stl
- link r_foot_9: geometry collision box size=0.5 0.2 0.05; visual mesh filename=r_foot.stl

File: res/benchmark/Atlas-contact-benchmark/mujoco/robot25.urdf (robot description, URDF)
Before this commit: robot drc_skeleton, 1102 links, 1100 joints
Links:
- link l_foot_0: geometry collision box size=0.5 0.2 0.05; visual mesh filename=l_foot.stl
- link l_foot_1: geometry collision box size=0.5 0.2 0.05; visual mesh filename=l_foot.stl
- link l_foot_10: geometry collision box size=0.5 0.2 0.05; visual mesh filename=l_foot.stl
- link l_foot_11: geometry collision box size=0.5 0.2 0.05; visual mesh filename=l_foot.stl
- link l_foot_12: geometry collision box size=0.5 0.2 0.05; visual mesh filename=l_foot.stl
- link l_foot_13: geometry collision box size=0.5 0.2 0.05; visual mesh filename=l_foot.stl
- link l_foot_14: geometry collision box size=0.5 0.2 0.05; visual mesh filename=l_foot.stl
- link l_foot_15: geometry collision box size=0.5 0.2 0.05; visual mesh filename=l_foot.stl
- link l_foot_16: geometry collision box size=0.5 0.2 0.05; visual mesh filename=l_foot.stl
- link l_foot_17: geometry collision box size=0.5 0.2 0.05; visual mesh filename=l_foot.stl
- link l_foot_18: geometry collision box size=0.5 0.2 0.05; visual mesh filename=l_foot.stl
- link l_foot_19: geometry collision box size=0.5 0.2 0.05; visual mesh filename=l_foot.stl
- link l_foot_2: geometry collision box size=0.5 0.2 0.05; visual mesh filename=l_foot.stl
- link l_foot_20: geometry collision box size=0.5 0.2 0.05; visual mesh filename=l_foot.stl
- link l_foot_21: geometry collision box size=0.5 0.2 0.05; visual mesh filename=l_foot.stl
- link l_foot_22: geometry collision box size=0.5 0.2 0.05; visual mesh filename=l_foot.stl
- link l_foot_23: geometry collision box size=0.5 0.2 0.05; visual mesh filename=l_foot.stl
- link l_foot_24: geometry collision box size=0.5 0.2 0.05; visual mesh filename=l_foot.stl
- link l_foot_3: geometry collision box size=0.5 0.2 0.05; visual mesh filename=l_foot.stl
- link l_foot_4: geometry collision box size=0.5 0.2 0.05; visual mesh filename=l_foot.stl
- link l_foot_5: geometry collision box size=0.5 0.2 0.05; visual mesh filename=l_foot.stl
- link l_foot_6: geometry collision box size=0.5 0.2 0.05; visual mesh filename=l_foot.stl
- link l_foot_7: geometry collision box size=0.5 0.2 0.05; visual mesh filename=l_foot.stl
- link l_foot_8: geometry collision box size=0.5 0.2 0.05; visual mesh filename=l_foot.stl
- link l_foot_9: geometry collision box size=0.5 0.2 0.05; visual mesh filename=l_foot.stl
- link r_foot_0: geometry collision box size=0.5 0.2 0.05; visual mesh filename=r_foot.stl
- link r_foot_1: geometry collision box size=0.5 0.2 0.05; visual mesh filename=r_foot.stl
- link r_foot_10: geometry collision box size=0.5 0.2 0.05; visual mesh filename=r_foot.stl
- link r_foot_11: geometry collision box size=0.5 0.2 0.05; visual mesh filename=r_foot.stl
- link r_foot_12: geometry collision box size=0.5 0.2 0.05; visual mesh filename=r_foot.stl
- link r_foot_13: geometry collision box size=0.5 0.2 0.05; visual mesh filename=r_foot.stl
- link r_foot_14: geometry collision box size=0.5 0.2 0.05; visual mesh filename=r_foot.stl
- link r_foot_15: geometry collision box size=0.5 0.2 0.05; visual mesh filename=r_foot.stl
- link r_foot_16: geometry collision box size=0.5 0.2 0.05; visual mesh filename=r_foot.stl
- link r_foot_17: geometry collision box size=0.5 0.2 0.05; visual mesh filename=r_foot.stl
- link r_foot_18: geometry collision box size=0.5 0.2 0.05; visual mesh filename=r_foot.stl
- link r_foot_19: geometry collision box size=0.5 0.2 0.05; visual mesh filename=r_foot.stl
- link r_foot_2: geometry collision box size=0.5 0.2 0.05; visual mesh filename=r_foot.stl
- link r_foot_20: geometry collision box size=0.5 0.2 0.05; visual mesh filename=r_foot.stl
- link r_foot_21: geometry collision box size=0.5 0.2 0.05; visual mesh filename=r_foot.stl
- link r_foot_22: geometry collision box size=0.5 0.2 0.05; visual mesh filename=r_foot.stl
- link r_foot_23: geometry collision box size=0.5 0.2 0.05; visual mesh filename=r_foot.stl
- link r_foot_24: geometry collision box size=0.5 0.2 0.05; visual mesh filename=r_foot.stl
- link r_foot_3: geometry collision box size=0.5 0.2 0.05; visual mesh filename=r_foot.stl
- link r_foot_4: geometry collision box size=0.5 0.2 0.05; visual mesh filename=r_foot.stl
- link r_foot_5: geometry collision box size=0.5 0.2 0.05; visual mesh filename=r_foot.stl
- link r_foot_6: geometry collision box size=0.5 0.2 0.05; visual mesh filename=r_foot.stl
- link r_foot_7: geometry collision box size=0.5 0.2 0.05; visual mesh filename=r_foot.stl
- link r_foot_8: geometry collision box size=0.5 0.2 0.05; visual mesh filename=r_foot.stl
- link r_foot_9: geometry collision box size=0.5 0.2 0.05; visual mesh filename=r_foot.stl

File: res/benchmark/Atlas-contact-benchmark/mujoco/robot4.urdf (robot description, URDF)
Before this commit: robot drc_skeleton, 178 links, 176 joints
Links:
- link l_foot_0: geometry collision box size=0.5 0.2 0.05; visual mesh filename=l_foot.stl
- link l_foot_1: geometry collision box size=0.5 0.2 0.05; visual mesh filename=l_foot.stl
- link l_foot_2: geometry collision box size=0.5 0.2 0.05; visual mesh filename=l_foot.stl
- link l_foot_3: geometry collision box size=0.5 0.2 0.05; visual mesh filename=l_foot.stl
- link r_foot_0: geometry collision box size=0.5 0.2 0.05; visual mesh filename=r_foot.stl
- link r_foot_1: geometry collision box size=0.5 0.2 0.05; visual mesh filename=r_foot.stl
- link r_foot_2: geometry collision box size=0.5 0.2 0.05; visual mesh filename=r_foot.stl
- link r_foot_3: geometry collision box size=0.5 0.2 0.05; visual mesh filename=r_foot.stl

File: res/benchmark/Atlas-contact-benchmark/mujoco/robot9.urdf (robot description, URDF)
Before this commit: robot drc_skeleton, 398 links, 396 joints
Links:
- link l_foot_0: geometry collision box size=0.5 0.2 0.05; visual mesh filename=l_foot.stl
- link l_foot_1: geometry collision box size=0.5 0.2 0.05; visual mesh filename=l_foot.stl
- link l_foot_2: geometry collision box size=0.5 0.2 0.05; visual mesh filename=l_foot.stl
- link l_foot_3: geometry collision box size=0.5 0.2 0.05; visual mesh filename=l_foot.stl
- link l_foot_4: geometry collision box size=0.5 0.2 0.05; visual mesh filename=l_foot.stl
- link l_foot_5: geometry collision box size=0.5 0.2 0.05; visual mesh filename=l_foot.stl
- link l_foot_6: geometry collision box size=0.5 0.2 0.05; visual mesh filename=l_foot.stl
- link l_foot_7: geometry collision box size=0.5 0.2 0.05; visual mesh filename=l_foot.stl
- link l_foot_8: geometry collision box size=0.5 0.2 0.05; visual mesh filename=l_foot.stl
- link r_foot_0: geometry collision box size=0.5 0.2 0.05; visual mesh filename=r_foot.stl
- link r_foot_1: geometry collision box size=0.5 0.2 0.05; visual mesh filename=r_foot.stl
- link r_foot_2: geometry collision box size=0.5 0.2 0.05; visual mesh filename=r_foot.stl
- link r_foot_3: geometry collision box size=0.5 0.2 0.05; visual mesh filename=r_foot.stl
- link r_foot_4: geometry collision box size=0.5 0.2 0.05; visual mesh filename=r_foot.stl
- link r_foot_5: geometry collision box size=0.5 0.2 0.05; visual mesh filename=r_foot.stl
- link r_foot_6: geometry collision box size=0.5 0.2 0.05; visual mesh filename=r_foot.stl
- link r_foot_7: geometry collision box size=0.5 0.2 0.05; visual mesh filename=r_foot.stl
- link r_foot_8: geometry collision box size=0.5 0.2 0.05; visual mesh filename=r_foot.stl

File: res/benchmark/Atlas-contact-benchmark/ode-rai-dart/robot.urdf (robot description, URDF)
Before this commit: robot drc_skeleton, 44 links, 43 joints
Links:
- link l_foot: geometry collision box size=0.5 0.15 0.05; visual mesh filename=l_foot.stl
- link r_foot: geometry collision box size=0.5 0.15 0.05; visual mesh filename=r_foot.stl
