Commit message: - rai data update - minor changes

File: res/benchmark/ANYmal-momentum-benchmark/bullet/robot.urdf (robot description, URDF)
Before this commit: robot anymal, 18 links, 17 joints
Joints:
- joint LF_HAA: limit lower=-6.28 upper=6.28 effort=80 velocity=15 -> (none); type revolute -> continuous
- joint LF_HFE: limit lower=-6.28 upper=6.28 effort=80 velocity=15 -> (none); type revolute -> continuous
- joint LF_KFE: limit lower=-6.28 upper=6.28 effort=80 velocity=15 -> (none); type revolute -> continuous
- joint LH_HAA: limit lower=-6.28 upper=6.28 effort=80 velocity=15 -> (none); type revolute -> continuous
- joint LH_HFE: limit lower=-6.28 upper=6.28 effort=80 velocity=15 -> (none); type revolute -> continuous
- joint LH_KFE: limit lower=-6.28 upper=6.28 effort=80 velocity=15 -> (none); type revolute -> continuous
- joint RF_HAA: limit lower=-6.28 upper=6.28 effort=80 velocity=15 -> (none); type revolute -> continuous
- joint RF_HFE: limit lower=-6.28 upper=6.28 effort=80 velocity=15 -> (none); type revolute -> continuous
- joint RF_KFE: limit lower=-6.28 upper=6.28 effort=80 velocity=15 -> (none); type revolute -> continuous
- joint RH_HAA: limit lower=-6.28 upper=6.28 effort=80 velocity=15 -> (none); type revolute -> continuous
- joint RH_HFE: limit lower=-6.28 upper=6.28 effort=80 velocity=15 -> (none); type revolute -> continuous
- joint RH_KFE: limit lower=-6.28 upper=6.28 effort=80 velocity=15 -> (none); type revolute -> continuous

File: res/benchmark/ANYmal-momentum-benchmark/mujoco/robot.urdf (robot description, URDF)
Before this commit: robot anymal, 28 links, 27 joints
Joints:
- joint LF_HAA_0: type revolute -> continuous
- joint LF_HFE_0: type revolute -> continuous
- joint LF_KFE_0: type revolute -> continuous
- joint LH_HAA_0: type revolute -> continuous
- joint LH_HFE_0: type revolute -> continuous
- joint LH_KFE_0: type revolute -> continuous
- joint RF_HAA_0: type revolute -> continuous
- joint RF_HFE_0: type revolute -> continuous
- joint RF_KFE_0: type revolute -> continuous
- joint RH_HAA_0: type revolute -> continuous
- joint RH_HFE_0: type revolute -> continuous
- joint RH_KFE_0: type revolute -> continuous

File: res/benchmark/ANYmal-momentum-benchmark/ode-rai-dart/robot.urdf (robot description, URDF)
Before this commit: robot anymal, 18 links, 17 joints
Joints:
- joint LF_HAA: limit lower=-6.28 upper=6.28 effort=80 velocity=15 -> (none); type revolute -> continuous
- joint LF_HFE: limit lower=-6.28 upper=6.28 effort=80 velocity=15 -> (none); type revolute -> continuous
- joint LF_KFE: limit lower=-6.28 upper=6.28 effort=80 velocity=15 -> (none); type revolute -> continuous
- joint LH_HAA: limit lower=-6.28 upper=6.28 effort=80 velocity=15 -> (none); type revolute -> continuous
- joint LH_HFE: limit lower=-6.28 upper=6.28 effort=80 velocity=15 -> (none); type revolute -> continuous
- joint LH_KFE: limit lower=-6.28 upper=6.28 effort=80 velocity=15 -> (none); type revolute -> continuous
- joint RF_HAA: limit lower=-6.28 upper=6.28 effort=80 velocity=15 -> (none); type revolute -> continuous
- joint RF_HFE: limit lower=-6.28 upper=6.28 effort=80 velocity=15 -> (none); type revolute -> continuous
- joint RF_KFE: limit lower=-6.28 upper=6.28 effort=80 velocity=15 -> (none); type revolute -> continuous
- joint RH_HAA: limit lower=-6.28 upper=6.28 effort=80 velocity=15 -> (none); type revolute -> continuous
- joint RH_HFE: limit lower=-6.28 upper=6.28 effort=80 velocity=15 -> (none); type revolute -> continuous
- joint RH_KFE: limit lower=-6.28 upper=6.28 effort=80 velocity=15 -> (none); type revolute -> continuous
