Commit message: mujoco anymal script fixed (ground thickness)

File: res/benchmark/ANYmal-PD-benchmark/mujoco/robot1.urdf (robot description, URDF)
Before this commit: robot anymal, 28 links, 26 joints
Links:
- link ground: geometry collision box size=100 100 10

File: res/benchmark/ANYmal-PD-benchmark/mujoco/robot100.urdf (robot description, URDF)
Before this commit: robot anymal, 2602 links, 2600 joints
Links:
- link ground: geometry collision box size=100 100 10

File: res/benchmark/ANYmal-PD-benchmark/mujoco/robot121.urdf (robot description, URDF)
Before this commit: robot anymal, 3148 links, 3146 joints
Links:
- link ground: geometry collision box size=100 100 10

File: res/benchmark/ANYmal-PD-benchmark/mujoco/robot144.urdf (robot description, URDF)
Before this commit: robot anymal, 3746 links, 3744 joints
Links:
- link ground: geometry collision box size=100 100 10

File: res/benchmark/ANYmal-PD-benchmark/mujoco/robot16.urdf (robot description, URDF)
Before this commit: robot anymal, 418 links, 416 joints
Links:
- link ground: geometry collision box size=100 100 10

File: res/benchmark/ANYmal-PD-benchmark/mujoco/robot169.urdf (robot description, URDF)
Before this commit: robot anymal, 4396 links, 4394 joints
Links:
- link ground: geometry collision box size=100 100 10

File: res/benchmark/ANYmal-PD-benchmark/mujoco/robot196.urdf (robot description, URDF)
Before this commit: robot anymal, 5098 links, 5096 joints
Links:
- link ground: geometry collision box size=100 100 10

File: res/benchmark/ANYmal-PD-benchmark/mujoco/robot25.urdf (robot description, URDF)
Before this commit: robot anymal, 652 links, 650 joints
Links:
- link ground: geometry collision box size=100 100 10

File: res/benchmark/ANYmal-PD-benchmark/mujoco/robot36.urdf (robot description, URDF)
Before this commit: robot anymal, 938 links, 936 joints
Links:
- link ground: geometry collision box size=100 100 10

File: res/benchmark/ANYmal-PD-benchmark/mujoco/robot4.urdf (robot description, URDF)
Before this commit: robot anymal, 106 links, 104 joints
Links:
- link ground: geometry collision box size=100 100 10

File: res/benchmark/ANYmal-PD-benchmark/mujoco/robot49.urdf (robot description, URDF)
Before this commit: robot anymal, 1276 links, 1274 joints
Links:
- link ground: geometry collision box size=100 100 10

File: res/benchmark/ANYmal-PD-benchmark/mujoco/robot64.urdf (robot description, URDF)
Before this commit: robot anymal, 1666 links, 1664 joints
Links:
- link ground: geometry collision box size=100 100 10

File: res/benchmark/ANYmal-PD-benchmark/mujoco/robot81.urdf (robot description, URDF)
Before this commit: robot anymal, 2108 links, 2106 joints
Links:
- link ground: geometry collision box size=100 100 10

File: res/benchmark/ANYmal-PD-benchmark/mujoco/robot9.urdf (robot description, URDF)
Before this commit: robot anymal, 236 links, 234 joints
Links:
- link ground: geometry collision box size=100 100 10
